File: SixEyes Follower PCB/SixEyes Follower PCB/SixEyes Follower PCB.kicad_sch (KiCad schematic)
At the start: 80 parts, among them J1 Conn_01x22_Socket, J10 Conn_01x08_Socket, J11 Conn_01x02, J12 Conn_01x02, J13 Conn_01x02, J14 Conn_01x02, J15 Conn_01x02, J16 JSTXH 4PIN to LEADER, J17 Conn_01x04, J18 Conn_01x04, J19 Conn_01x04, J1_MOTOR JST-XH-6-STEPPER, J2 Conn_01x22_Socket, J20 Conn_01x04, J21 Conn_01x03, J22 Conn_01x03, J23 Conn_01x03, J2_MOTOR JST-XH-6-STEPPER, J3 Conn_01x08_Socket, J3_MOTOR JST-XH-6-STEPPER, J4 Conn_01x08_Socket, J4_MOTOR JST-XH-6-STEPPER, J5 Conn_01x08_Socket, J6 Conn_01x08_Socket, J7 Conn_01x08_Socket, J8 Conn_01x08_Socket, J9 Conn_01x08_Socket, U1A ESP32-S3-SOCK-LEFT, U1B ESP32-S3-SOCK-RIGHT, U2 TMC2209-J1-BASE, U3 TMC2209-J2-SHOULDER-A, U4 TMC2209-J3-SHOULDER-B, U5 TMC2209-J4-ELBOW

Commit message: refactor: flatten sixeyes/ to root, add KiCad PCB project, fix JSON pipeline, fix safety bitmask, implement ROS2 nodes, update docs
- Flatten sixeyes/ wrapper: firmware/, ros2_ws/, tools/, simulation/, hardware_assets/ now at repo root
- Merge sixeyes/docs/ into docs/ (safety.md, protocols/uart_protocol.md)
- Add KiCad follower PCB project files (.kicad_pro, .kicad_prl, fp-lib-table, custom footprints, design_inputs/)
- Update .gitignore: exclude KiCad .history/ and *-backups/ directories
- Fix UartJsonParser pipeline: init() now called in MessageRouter::init(), update() ticked each control loop iteration
- Add JOINT_STATE (type 8) to MessageType enum, parse block, struct, and TeleoperationHandler callback
- Fix FaultManager: uint32_t bitmask supports simultaneous faults, add clearFault(f)
- Fix SafetyTask: isSafeToOperate() checks both HeartbeatMonitor and ROS2 alive; use SAFETY_HEARTBEAT_TIMEOUT_MS constant
- Fix main.cpp: UsbCDC::update() now called in loop()
- Fix MotorControlScheduler: 500 Hz (was 400 Hz), UartJsonParser::update() added to control loop
- Implement ROS2 nodes: usb_bridge_node, safety_node, camera_node, joint_state_node
- Update docs: FIRMWARE_FEATURE_INVENTORY, TELEOPERATION_MODE_ARCHITECTURE, JSON_MESSAGE_PROTOCOL, PROJECT_SCOPE_AND_REPO_MAP, README
Parts:
- removed C1: 470uF/35V, Capacitor_THT:CP_Radial_D10.0mm_P5.00mm, symbol SixEyes:CP_RADIAL
- removed C10, C11, C13, C3, C5, C7, C8, C9: 100nF, Capacitor_THT:C_Disc_D5.0mm_W2.5mm_P5.00mm, symbol SixEyes:C_DISC
- removed C12: 10uF/10V, Capacitor_THT:CP_Radial_D5.0mm_P2.00mm, symbol SixEyes:CP_RADIAL
- removed C2: 1uF/50V, Capacitor_THT:C_Disc_D5.0mm_W2.5mm_P5.00mm, symbol SixEyes:C_DISC
- removed C4: 1000uF/16V, Capacitor_THT:CP_Radial_D10.0mm_P5.00mm, symbol SixEyes:CP_RADIAL
- removed C6: 220uF/10V, Capacitor_THT:CP_Radial_D8.0mm_P3.50mm, symbol SixEyes:CP_RADIAL
- removed H_SD1: HDR-1x06-SD-SPI, Connector_PinSocket_2.54mm:PinSocket_1x06_P2.54mm_Vertical, symbol SixEyes:HDR_1x06_SD_SPI
- removed H_UART1: HDR-1x04-UART, Connector_PinHeader_2.54mm:PinHeader_1x04_P2.54mm_Vertical, symbol SixEyes:HDR_1x04_UART
- removed J1_MOTOR, J2_MOTOR, J3_MOTOR, J4_MOTOR: JST-XH-6-STEPPER, Connector_JST:JST_XH_B6B-XH-A_1x06_P2.50mm_Vertical, symbol SixEyes:JST6_STEPPER_4USED
- removed J_PWR1: PWR-IN-24V, TerminalBlock:TerminalBlock_bornier-2_P5.08mm, symbol SixEyes:TERMINAL_2P_24V
- removed J_PWR2: 24V-OUT-BUCK3V3-IN, TerminalBlock:TerminalBlock_bornier-2_P5.08mm, symbol SixEyes:TERMINAL_2P_24V
- removed J_PWR3: 24V-OUT-BUCK6V6-IN, TerminalBlock:TerminalBlock_bornier-2_P5.08mm, symbol SixEyes:TERMINAL_2P_24V
- removed J_PWR4: BUCK3V3-OUT-IN, TerminalBlock:TerminalBlock_bornier-2_P5.08mm, symbol SixEyes:TERMINAL_2P_24V
- removed J_PWR5: BUCK6V6-OUT-IN, TerminalBlock:TerminalBlock_bornier-2_P5.08mm, symbol SixEyes:TERMINAL_2P_24V
- removed J_SERVO1, J_SERVO2, J_SERVO3: JST-XH-3-SERVO, Connector_JST:JST_XH_B3B-XH-A_1x03_P2.50mm_Vertical, symbol SixEyes:JST3_SERVO
- removed R1, R2, R3, R4: 4.7k, Resistor_THT:R_Axial_DIN0207_L6.3mm_D2.5mm_P7.62mm_Horizontal, symbol SixEyes:R_AXIAL
- removed R10, R11, R9: 100k, Resistor_THT:R_Axial_DIN0207_L6.3mm_D2.5mm_P7.62mm_Horizontal, symbol SixEyes:R_AXIAL
- removed R12, R13: 220R DNI, Resistor_THT:R_Axial_DIN0207_L6.3mm_D2.5mm_P7.62mm_Horizontal, symbol SixEyes:R_AXIAL
- removed R14, R15, R16, R17: 33R DNI, Resistor_THT:R_Axial_DIN0207_L6.3mm_D2.5mm_P7.62mm_Horizontal, symbol SixEyes:R_AXIAL
- removed R5, R6, R7, R8: 0R DNI, Resistor_THT:R_Axial_DIN0207_L6.3mm_D2.5mm_P7.62mm_Horizontal, symbol SixEyes:R_AXIAL
- removed TP1: TP_EN_ALL, TestPoint:TestPoint_Pad_D1.5mm, symbol SixEyes:TESTPOINT_1P
- removed TP2: TP_PDN_J1, TestPoint:TestPoint_Pad_D1.5mm, symbol SixEyes:TESTPOINT_1P
- removed TP3: TP_PDN_J2, TestPoint:TestPoint_Pad_D1.5mm, symbol SixEyes:TESTPOINT_1P
- removed TP4: TP_PDN_J3, TestPoint:TestPoint_Pad_D1.5mm, symbol SixEyes:TESTPOINT_1P
- removed TP5: TP_PDN_J4, TestPoint:TestPoint_Pad_D1.5mm, symbol SixEyes:TESTPOINT_1P
- removed TP6: TP_UART_RX, TestPoint:TestPoint_Pad_D1.5mm, symbol SixEyes:TESTPOINT_1P
- removed TP7: TP_UART_TX, TestPoint:TestPoint_Pad_D1.5mm, symbol SixEyes:TESTPOINT_1P
- removed U1A: ESP32-S3-SOCK-LEFT, Connector_PinSocket_2.54mm:PinSocket_1x19_P2.54mm_Vertical, symbol SixEyes:ESP32_S3_SOCK_LEFT_1x19
- removed U1B: ESP32-S3-SOCK-RIGHT, Connector_PinSocket_2.54mm:PinSocket_1x19_P2.54mm_Vertical, symbol SixEyes:ESP32_S3_SOCK_RIGHT_1x19
- removed U2: TMC2209-J1-BASE, Connector_PinSocket_2.54mm:PinSocket_2x08_P2.54mm_Vertical, symbol SixEyes:TMC2209_DEVBOARD_2x08
- removed U3: TMC2209-J2-SHOULDER-A, Connector_PinSocket_2.54mm:PinSocket_2x08_P2.54mm_Vertical, symbol SixEyes:TMC2209_DEVBOARD_2x08
- removed U4: TMC2209-J3-SHOULDER-B, Connector_PinSocket_2.54mm:PinSocket_2x08_P2.54mm_Vertical, symbol SixEyes:TMC2209_DEVBOARD_2x08
- removed U5: TMC2209-J4-ELBOW, Connector_PinSocket_2.54mm:PinSocket_2x08_P2.54mm_Vertical, symbol SixEyes:TMC2209_DEVBOARD_2x08
- added C1: 470 uF, Capacitor_THT:CP_Radial_D10.0mm_P5.00mm, symbol Device:C
- added C10, C11, C13, C18, C19, C20, C24, C25, C3, C5, C7, C8, C9: 100 nF, Capacitor_THT:C_Disc_D5.0mm_W2.5mm_P5.00mm, symbol Device:C
- added C12, C14, C15, C16, C17, C21, C22, C23: 10 uF, Capacitor_THT:CP_Radial_D8.0mm_P3.50mm, symbol Device:C
- added C4: 1000 uF, Capacitor_THT:CP_Radial_D10.0mm_P5.00mm, symbol Device:C
- added C6: 220 uF, Capacitor_THT:C_Disc_D5.0mm_W2.5mm_P5.00mm, symbol Device:C
- added J24: DUPONT 7PIN TO SDREADER, Connector_PinSocket_2.54mm:PinSocket_1x07_P2.54mm_Vertical, symbol Connector_Generic:Conn_01x07
- added R1, R2, R3, R4: 4.7 k, Resistor_THT:R_Axial_DIN0207_L6.3mm_D2.5mm_P7.62mm_Horizontal, symbol Device:R
- added R10, R11, R9: 100k, Resistor_THT:R_Axial_DIN0207_L6.3mm_D2.5mm_P7.62mm_Horizontal, symbol Device:R
- added R12, R13, R14, R15, R16, R17: 220, Resistor_THT:R_Axial_DIN0207_L6.3mm_D2.5mm_P7.62mm_Horizontal, symbol Device:R
- J1, J2: footprint (none) -> Connector_PinSocket_2.54mm:PinSocket_1x22_P2.54mm_Vertical
- J10, J3, J4, J5, J6, J7, J8, J9: footprint (none) -> Connector_PinSocket_2.54mm:PinSocket_1x08_P2.54mm_Vertical
- J11, J12, J13, J14, J15: footprint (none) -> TerminalBlock_Phoenix:TerminalBlock_Phoenix_MKDS-1,5-2_1x02_P5.00mm_Horizontal
- J16, J17, J18, J19, J20: footprint (none) -> Connector_JST:JST_XH_B4B-XH-A_1x04_P2.50mm_Vertical
- J21, J22, J23: footprint (none) -> Connector_JST:JST_XH_B3B-XH-A_1x03_P2.50mm_Vertical
Connections:
- net TMC2209 J1 A1 is gone; now on net J1_MOTOR_PIN3 (B1): J17.3 (Pin_3)
- net TMC2209 J1 A2 is gone; now on net J1_MOTOR_PIN2 (A1): J17.2 (Pin_2)
- net TMC2209 J1 B1 is gone; now on net J1_MOTOR_PIN1 (A2): J17.1 (Pin_1)
- net TMC2209 J1 B2 is gone; now on net J1_MOTOR_PIN4 (B2): J17.4 (Pin_4)
- net TMC2209 J2 A1 is gone; now on net J2_MOTOR_PIN3 (B1): J18.3 (Pin_3)
- net TMC2209 J2 A2 is gone; now on net J2_MOTOR_PIN2 (A1): J18.2 (Pin_2)
- net TMC2209 J2 B1 is gone; now on net J2_MOTOR_PIN1 (A2): J18.1 (Pin_1)
- net TMC2209 J2 B2 is gone; now on net J2_MOTOR_PIN4 (B2): J18.4 (Pin_4)
- net +24V_MOTOR: now also J10.1 (Pin_1), J11.1 (Pin_1), J12.1 (Pin_1), J13.2 (Pin_2), J4.1 (Pin_1), J6.1 (Pin_1), J8.1 (Pin_1), C1.1, C14.1, C15.1, C16.1, C17.1, C18.1, C19.1, C20.1, C3.1
- net +3V3_LOGIC: now also J1.1 (3V3), J1.2 (Pin_2), J10.7 (Pin_7), J14.1 (Pin_1), J4.7 (Pin_7), J6.7 (Pin_7), J8.7 (Pin_7), C10.1, C11.2, C12.2, C13.2, C6.1, C7.1, C8.1, C9.1, J24.7 (Pin_7), R1.1, R2.1, R3.1, R4.1
- net +6V6_SERVO: now also J15.1 (Pin_1), J21.2 (Pin_2), J22.2 (Pin_2), J23.2 (Pin_2), C21.2, C22.2, C23.2, C24.2, C25.2, C4.1, C5.2
- net DIR_J1: now also J1.17 (Pin_17), J3.8 (Pin_8)
- net DIR_J2: now also J1.12 (Pin_12), J5.8 (Pin_8)
- net DIR_J3: now also J1.7 (Pin_7), J7.8 (Pin_8)
- net DIR_J4: now also J1.4 (Pin_4), J9.8 (Pin_8)
- net EN_ALL: now also J1.20 (Pin_20), J3.1 (Pin_1), J5.1 (Pin_1), J7.1 (Pin_1), J9.1 (Pin_1)
- net GND: now also J1.22 (Pin_22), J10.2 (Pin_2), J10.8 (Pin_8), J11.2 (Pin_2), J12.2 (Pin_2), J13.1 (Pin_1), J14.2 (Pin_2), J15.2 (Pin_2), J2.1 (Pin_1), J2.21 (Pin_21), J2.22 (Pin_22), J21.1 (Pin_1), J22.1 (Pin_1), J23.1 (Pin_1), J4.2 (Pin_2), J4.8 (Pin_8), J6.2 (Pin_2), J6.8 (Pin_8), J8.2 (Pin_2), J8.8 (Pin_8), C1.2, C10.2, C11.1, C12.1, C13.1, C14.2, C15.2, C16.2, C17.2, C18.2, C19.2, C20.2, C21.1, C22.1, C23.1, C24.1, C25.1, C3.2, C4.2, C5.1, C6.2, C7.2, C8.2, C9.2, J24.6 (Pin_6), R10.2, R11.2, R9.2
- net PDN_J1: now also J1.19 (Pin_19), J3.4 (Pin_4), R4.2
- net PDN_J2: now also J1.16 (Pin_16), J5.4 (Pin_4), R3.2
- net PDN_J3: now also J1.9 (Pin_9), J7.4 (Pin_4), R2.2
- net PDN_J4: now also J1.6 (Pin_6), J9.4 (Pin_4), R1.2
- net SD_CS: now also J2.10 (Pin_10), J24.5 (Pin_5), R17.1, R17.2
- net SD_MISO: now also J2.11 (Pin_11), J24.2 (Pin_2), R14.1, R14.2
- net SD_MOSI: now also J2.13 (Pin_13), J24.4 (Pin_4), R16.1, R16.2
- net SD_SCK: now also J2.12 (Pin_12), J24.3 (Pin_3), R15.1, R15.2
- net SERVO_GRIPPER: now also J2.6 (Pin_6), J23.3 (Pin_3), R11.1
- net SERVO_WRIST_PITCH: now also J2.8 (Pin_8), J21.3 (Pin_3), R9.1
- net SERVO_WRIST_YAW: now also J2.7 (Pin_7), J22.3 (Pin_3), R10.1
- net STEP_J1: now also J1.18 (Pin_18), J3.7 (Pin_7)
- net STEP_J2: now also J1.15 (Pin_15), J5.7 (Pin_7)
- net STEP_J3: now also J1.8 (Pin_8), J7.7 (Pin_7)
- net STEP_J4: now also J1.5 (Pin_5), J9.7 (Pin_7)
- net UART_LEADER_RX: now also J1.11 (Pin_11), R12.1, R12.2
- net UART_LEADER_TX: now also J1.10 (Pin_10), R13.1, R13.2
- net J2_MOTOR_PIN1 (A2): now reaches J6.3 (Pin_3)
- net J2_MOTOR_PIN2 (A1): now reaches J6.4 (Pin_4)
- net J2_MOTOR_PIN3 (B1): now reaches J6.5 (Pin_5)
- net J2_MOTOR_PIN4 (B2): now reaches J6.6 (Pin_6)
- net J3_MOTOR_PIN1 (A2): now reaches J8.3 (Pin_3)
- net J3_MOTOR_PIN1 (A2): now also J19.1 (Pin_1)
- net J3_MOTOR_PIN2 (A1): now reaches J8.4 (Pin_4)
- net J3_MOTOR_PIN2 (A1): now also J19.2 (Pin_2)
- net J3_MOTOR_PIN3 (B1): now reaches J8.5 (Pin_5)
- net J3_MOTOR_PIN3 (B1): now also J19.3 (Pin_3)
- net J3_MOTOR_PIN4 (B2): now reaches J8.6 (Pin_6)
- net J3_MOTOR_PIN4 (B2): now also J19.4 (Pin_4)
- net J1_MOTOR_PIN1 (A2): now reaches J4.3 (Pin_3)
- net J1_MOTOR_PIN2 (A1): now reaches J4.4 (Pin_4)
- net J1_MOTOR_PIN3 (B1): now reaches J4.5 (Pin_5)
- net J1_MOTOR_PIN4 (B2): now reaches J4.6 (Pin_6)
- net J4_MOTOR_PIN1 (A2): now reaches J20.1 (Pin_1)
- net J4_MOTOR_PIN1 (A2): now also J10.3 (Pin_3)
- net J4_MOTOR_PIN2 (A1): now reaches J20.2 (Pin_2)
- net J4_MOTOR_PIN2 (A1): now also J10.4 (Pin_4)
- net J4_MOTOR_PIN3 (B1): now reaches J20.3 (Pin_3)
- net J4_MOTOR_PIN3 (B1): now also J10.5 (Pin_5)
- net J4_MOTOR_PIN4 (B2): now reaches J20.4 (Pin_4)
- net J4_MOTOR_PIN4 (B2): now also J10.6 (Pin_6)
- net OLED1: now reaches J2.2 (Pin_2)
- net OLED2: now reaches J2.3 (Pin_3)
- net OLED3: now reaches J2.4 (Pin_4)
- net OLED4: now reaches J2.5 (Pin_5)
- net SD_CD: now reaches J2.9 (Pin_9)
- net SD_CD: now also J24.1 (Pin_1)
Other:
- moved on the sheet: J1, J11, J12, J13, J14, J15, J16, J17, J18, J19, J2, J21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
